Commit message: added hiqp controller launcher, fixed joint offsets to avoid singularity at start

File: gbot_description/urdf/3dof_planar.xacro (robot description, xacro)
@@ -59,9 +59,9 @@
     <joint name="${arm_id}_joint1" type="revolute">
       <safety_controller k_position="100.0" k_velocity="40.0" soft_lower_limit="-2.8973" soft_upper_limit="2.8973"/>
-      <origin rpy="0 0 0" xyz="0 0 0.05"/>
+      <origin rpy="0 0 ${pi/4}" xyz="0 0 0.05"/>
       <parent link="${arm_id}_link0"/>
       <child link="${arm_id}_link1"/>
       <axis xyz="0 0 1"/>
-      <limit effort="150" lower="-2.8973" upper="2.8973" velocity="2.1750"/>
+      <limit effort="150" lower="-2" upper="2" velocity="2.1750"/>
       <!-- for simulation -->
       <dynamics damping="${joint_damping}" friction="0.546"/>
@@ -91,9 +91,9 @@
     <joint name="${arm_id}_joint2" type="revolute">
       <safety_controller k_position="100.0" k_velocity="40.0" soft_lower_limit="-2.8973" soft_upper_limit="2.8973"/>
-      <origin rpy="0 0 0" xyz="${link1_length} 0 0"/>
+      <origin rpy="0 0 ${-pi/8}" xyz="${link1_length} 0 0"/>
       <parent link="${arm_id}_link1"/>
       <child link="${arm_id}_link2"/>
       <axis xyz="0 0 1"/>
-      <limit effort="150" lower="-2.8973" upper="2.8973" velocity="2.1750"/>
+      <limit effort="150" lower="-2" upper="2" velocity="2.1750"/>
       <!-- for simulation -->
       <dynamics damping="${joint_damping}" friction="0.546"/>
@@ -123,9 +123,9 @@
     <joint name="${arm_id}_joint3" type="revolute">
       <safety_controller k_position="100.0" k_velocity="40.0" soft_lower_limit="-2.8973" soft_upper_limit="2.8973"/>
-      <origin rpy="0 0 0" xyz="${link2_length} 0 0"/>
+      <origin rpy="0 0 ${-pi/8}" xyz="${link2_length} 0 0"/>
       <parent link="${arm_id}_link2"/>
       <child link="${arm_id}_link3"/>
       <axis xyz="0 0 1"/>
-      <limit effort="150" lower="-2.8973" upper="2.8973" velocity="2.1750"/>
+      <limit effort="150" lower="-2" upper="2" velocity="2.1750"/>
       <!-- for simulation -->
       <dynamics damping="${joint_damping}" friction="0.546"/>

Commit message: pulled in the ycb objects here

File: gbot_description/urdf/3dof_planar.xacro (robot description, xacro)
@@ -53,5 +53,6 @@
         <origin xyz="${link1_length/2} 0.0 0.0" rpy="0 0 0" />
         <mass value="1.0" />
-        <inertia izz="0.02" ixy="0.0" ixz="0.0" iyy="0.02" iyz="0.0" ixx="0.0002" />
+        <!--inertia izz="0.02" ixy="0.0" ixz="0.0" iyy="0.02" iyz="0.0" ixx="0.0002" /-->
+        <inertia izz="0.0" ixy="0.0" ixz="0.0" iyy="0.0" iyz="0.0" ixx="0.0" />
       </inertial>
       <!-- end for simulation -->
@@ -85,5 +86,6 @@
         <origin xyz="${link2_length/2} 0.0 0.0" rpy="0 0 0" />
         <mass value="0.6" />
-        <inertia izz="0.00456" ixy="0.0" ixz="0.0" iyy="0.00456" iyz="0.0" ixx="0.0001" />
+        <!--inertia izz="0.00456" ixy="0.0" ixz="0.0" iyy="0.00456" iyz="0.0" ixx="0.0001" /-->
+        <inertia izz="0.0" ixy="0.0" ixz="0.0" iyy="0.0" iyz="0.0" ixx="0.0" />
       </inertial>
       <!-- end for simulation -->
@@ -117,5 +119,6 @@
         <origin xyz="${link3_length/2} 0.0 0.0" rpy="0 0 0" />
         <mass value="0.3" />
-        <inertia izz="0.00103" ixy="0.0" ixz="0.0" iyy="0.00103" iyz="0.0" ixx="0.00006" />
+        <!--inertia izz="0.00103" ixy="0.0" ixz="0.0" iyy="0.00103" iyz="0.0" ixx="0.00006" /-->
+        <inertia izz="0.0" ixy="0.0" ixz="0.0" iyy="0.0" iyz="0.0" ixx="0.0" />
       </inertial>
       <!-- end for simulation -->

Commit message: fixing joint limits and safety controllers, adding limit tasks in hiqp

File: gbot_description/urdf/3dof_planar.xacro (robot description, xacro)
@@ -59,10 +59,10 @@
     </link>
     <joint name="${arm_id}_joint1" type="revolute">
-      <safety_controller k_position="100.0" k_velocity="40.0" soft_lower_limit="-2.8973" soft_upper_limit="2.8973"/>
+      <safety_controller k_position="100.0" k_velocity="40.0" soft_lower_limit="-1.9" soft_upper_limit="1.9"/>
       <origin rpy="0 0 ${pi/4}" xyz="0 0 0.05"/>
       <parent link="${arm_id}_link0"/>
       <child link="${arm_id}_link1"/>
       <axis xyz="0 0 1"/>
-      <limit effort="150" lower="-2" upper="2" velocity="2.1750"/>
+      <limit effort="15" lower="-2" upper="2" velocity="2.1750"/>
       <!-- for simulation -->
       <dynamics damping="${joint_damping}" friction="0.546"/>
@@ -92,10 +92,10 @@
     </link>
     <joint name="${arm_id}_joint2" type="revolute">
-      <safety_controller k_position="100.0" k_velocity="40.0" soft_lower_limit="-2.8973" soft_upper_limit="2.8973"/>
+      <safety_controller k_position="100.0" k_velocity="40.0" soft_lower_limit="-1.9" soft_upper_limit="1.9"/>
       <origin rpy="0 0 ${-pi/8}" xyz="${link1_length} 0 0"/>
       <parent link="${arm_id}_link1"/>
       <child link="${arm_id}_link2"/>
       <axis xyz="0 0 1"/>
-      <limit effort="150" lower="-2" upper="2" velocity="2.1750"/>
+      <limit effort="15" lower="-2" upper="2" velocity="2.1750"/>
       <!-- for simulation -->
       <dynamics damping="${joint_damping}" friction="0.546"/>
@@ -125,10 +125,10 @@
     </link>
     <joint name="${arm_id}_joint3" type="revolute">
-      <safety_controller k_position="100.0" k_velocity="40.0" soft_lower_limit="-2.8973" soft_upper_limit="2.8973"/>
+      <safety_controller k_position="100.0" k_velocity="40.0" soft_lower_limit="-1.9" soft_upper_limit="1.9"/>
       <origin rpy="0 0 ${-pi/8}" xyz="${link2_length} 0 0"/>
       <parent link="${arm_id}_link2"/>
       <child link="${arm_id}_link3"/>
       <axis xyz="0 0 1"/>
-      <limit effort="150" lower="-2" upper="2" velocity="2.1750"/>
+      <limit effort="15" lower="-2" upper="2" velocity="2.1750"/>
       <!-- for simulation -->
       <dynamics damping="${joint_damping}" friction="0.546"/>
